Commit message: fix(urdf-generator): enable MuJoCo 3D visualization and fix model loading
This PR fixes multiple issues preventing the URDF Generator from launching
models and rendering them in MuJoCo 3D view:

**Path and Import Fixes:**
- Fix model paths in models.yaml (add missing `src/` prefix)
- Fix URDF_GENERATOR_SCRIPT and C3D_VIEWER_SCRIPT paths in constants.py
- Fix `model.repo_path` -> `model.path` attribute access in golf_launcher.py
- Add PYTHONPATH to subprocess environment for module resolution
- Add sys.path setup in launcher scripts for standalone execution

**MuJoCo Integration Fixes:**
- Import MuJoCo BEFORE Qt to avoid DLL conflicts on Windows
- Fix Renderer parameter order (height, width) not (width, height)
- Fix GRAVITY_M_S2 PhysicalConstant to float conversion for MJCF
- Add preprocessing to fix zero/small mass and inertia values
- Use model's offscreen dimensions for framebuffer compatibility

**Bundled Assets:**
- Fix URDF mesh paths from `package://` URLs to relative paths
- Update bundled_assets module with proper path setup
- Load models from bundled assets instead of attempting downloads

Co-Authored-By: Claude Opus 4.5 <noreply@anthropic.com>

File: src/tools/urdf_generator/bundled_assets/human_models/human_subject_with_meshes/model.urdf (robot description, URDF)
Before this commit: robot HumanModel, 93 links, 92 joints
Links:
- link Head: geometry collision sphere radius=0.1105; visual mesh filename=meshes/Head.stl scale=1.03030303 1.03030303 1.03030303
- link LeftFoot: geometry collision box size=0.2584 0.0935 0.0663; visual mesh filename=meshes/LeftFoot.stl scale=1.03030303 1.03030303 1.03030303
- link LeftForeArm: geometry collision cylinder length=0.24819999999999998 radius=0.0275; visual mesh filename=meshes/LeftExtCarp.stl scale=0.61111111 0.61111111 1.03030303
- link LeftHand: geometry collision box size=0.072 0.1836 0.025; visual mesh filename=meshes/LeftHand.stl scale=0.9 1.03030303 0.55555556
- link LeftLowerLeg: geometry collision cylinder length=0.41819999999999996 radius=0.045; visual mesh filename=meshes/LeftGasLat.stl scale=0.7826087 0.7826087 1.03030303
- link LeftShoulder: geometry collision cylinder length=0.14676666666666668 radius=0.029; visual mesh filename=meshes/LeftShoulder.stl scale=0.64444444 0.64444444 1.03030303
- link LeftToe: geometry collision box size=0.002584 0.0935 0.0663; visual mesh filename=meshes/LeftToe.stl scale=1.03030303 1.03030303 1.03030303
- link LeftUpperArm: geometry collision cylinder length=0.3162 radius=0.029; visual mesh filename=meshes/LeftBicBrac.stl scale=0.64444444 0.64444444 1.03030303
- link LeftUpperLeg: geometry collision cylinder length=0.4165 radius=0.0625; visual mesh filename=meshes/LeftBicFem.stl scale=0.83333333 0.83333333 1.03030303
- link LowerTrunk: geometry collision box size=0.175 0.2958 0.17; visual mesh filename=meshes/LowerTrunk.stl scale=0.58333333 1.03030303 1.03030303
- link Neck: geometry collision cylinder length=0.08839999999999999 radius=0.0475; visual mesh filename=meshes/Neck.stl scale=0.73076923 0.73076923 1.03030303
- link Pelvis: geometry collision box size=0.175 0.3247 0.1326; visual mesh filename=meshes/Pelvis.stl scale=0.58333333 1.03030303 1.03030303
- link RightFoot: geometry collision box size=0.2584 0.0935 0.0663; visual mesh filename=meshes/RightFoot.stl scale=1.03030303 1.03030303 1.03030303
- link RightForeArm: geometry collision cylinder length=0.24819999999999998 radius=0.0275; visual mesh filename=meshes/RightExtCarp.stl scale=0.61111111 0.61111111 1.03030303
- link RightHand: geometry collision box size=0.072 0.1836 0.025; visual mesh filename=meshes/RightHand.stl scale=0.9 1.03030303 0.55555556
- link RightLowerLeg: geometry collision cylinder length=0.41819999999999996 radius=0.045; visual mesh filename=meshes/RightGasLat.stl scale=0.7826087 0.7826087 1.03030303
- link RightShoulder: geometry collision cylinder length=0.14676666666666668 radius=0.029; visual mesh filename=meshes/RightShoulder.stl scale=0.64444444 0.64444444 1.03030303
- link RightToe: geometry collision box size=0.002584 0.0935 0.0663; visual mesh filename=meshes/RightToe.stl scale=1.03030303 1.03030303 1.03030303
- link RightUpperArm: geometry collision cylinder length=0.3162 radius=0.029; visual mesh filename=meshes/RightBicBrac.stl scale=0.64444444 0.64444444 1.03030303
- link RightUpperLeg: geometry collision cylinder length=0.4165 radius=0.0625; visual mesh filename=meshes/RightBicFem.stl scale=0.83333333 0.83333333 1.03030303
- link UpperTrunk: geometry collision box size=0.175 0.14676667 0.187; visual mesh filename=meshes/UpperTrunk.stl scale=0.58333333 1.03030303 1.03030303
