Commit message: feat(model-converter): cross-engine URDF and MJCF exporters from canonical spec (#9965) (#9982)
* feat(model-converter): cross-engine URDF and MJCF exporters from canonical spec (#9965)

* fix(model-converter): add architecture budget exceptions and suite markers

* fix(model-converter): move model_converter from tools to src/tools (#9965)

* fix(model-converter): correct REPO_ROOT parent depth in build_models.py

* fix(model-converter): resolve Law of Demeter violations in exporters (#9965)

* fix(model-converter): update architecture budget exception paths to src/tools (#9965)

* refactor(model-converter): extract shared XML joint helpers in URDF exporter

* fix(model-converter): register model_converter in registry exclusions (#9965)

* fix(security): annotate element creation imports for semgrep in model_converter (#9965)

---------

Co-authored-by: d-sorgcodexagent <d-sorgcodexagent@users.noreply.github.com>
Co-authored-by: github-actions[bot] <41898282+github-actions[bot]@users.noreply.github.com>

File: src/engines/physics_engines/pinocchio/models/generated/golfer.urdf (robot description, URDF)
Before this commit: robot golfer, 47 links, 46 joints
Links:
- added link head, mass 5; visual sphere radius=0.12
- link club_head: mass 0.2 -> 0.23
- link club_shaft: mass 0.05 -> 0.12; geometry visual cylinder length=0.5 radius=0.015
- link forearm_left: mass 1.18 -> 1.5; geometry visual cylinder length=0.13 radius=0.045
- link forearm_right: mass 1.18 -> 1.5; geometry visual cylinder length=0.13 radius=0.045
- link hand_left: mass 0.61 -> 0.5; geometry visual cylinder length=0.095 radius=0.04
- link hand_right: mass 0.61 -> 0.5; geometry visual cylinder length=0.095 radius=0.04
- link left_shank: geometry visual cylinder length=0.215 radius=0.05
- link left_thigh: geometry visual cylinder length=0.215 radius=0.06
- link lumbar1: mass 2.0 -> 2; geometry visual cylinder length=0.12 radius=0.08
- link lumbar2: mass 2.0 -> 2; geometry visual cylinder length=0.12 radius=0.08
- link lumbar3: mass 2.0 -> 2; geometry visual cylinder length=0.12 radius=0.08
- link mid_hands: mass 0.001 -> None
- link pelvis: geometry visual cylinder length=0.2 radius=0.15
- link right_shank: geometry visual cylinder length=0.215 radius=0.05
- link right_thigh: geometry visual cylinder length=0.215 radius=0.06
- link thorax1: mass 1.5 -> 6; geometry visual cylinder length=0.1 radius=0.08
- link thorax2: mass 1.5 -> 6; geometry visual cylinder length=0.1 radius=0.08
- link thorax3: mass 1.5 -> 6; geometry visual cylinder length=0.1 radius=0.08
- link upper_arm_left: mass 1.98 -> 2.5; geometry visual cylinder length=0.14 radius=0.05
- link upper_arm_right: mass 1.98 -> 2.5; geometry visual cylinder length=0.14 radius=0.05
Joints:
- added joint thorax3_to_head: type fixed, parent thorax3, child head, origin xyz=0 0 0.15 rpy=0 0 0
- joint club_shaft_to_club_head: origin xyz=0.0 0.0 -0.5 rpy=0.0 0.0 0.0 -> xyz=0 0 -0.5 rpy=0 0 0
- joint forearm_left_to_hand_left_intermediate: origin xyz=0.0 0.0 -0.19 rpy=0.0 0.0 0.0 -> xyz=0 0 -0.19 rpy=0 0 0
- joint forearm_right_to_hand_right_intermediate: origin xyz=0.0 0.0 -0.19 rpy=0.0 0.0 0.0 -> xyz=0 0 -0.19 rpy=0 0 0
- joint hand_left_to_fingers_left: limit lower=0.0 upper=1.57 effort=1000.0 velocity=10.0 -> lower=0 upper=1.57 effort=1000.0 velocity=10.0; origin xyz=0.0 0.0 -0.05 rpy=0.0 0.0 0.0 -> xyz=0 0 -0.05 rpy=0 0 0
- joint hand_right_to_fingers_right: limit lower=0.0 upper=1.57 effort=1000.0 velocity=10.0 -> lower=0 upper=1.57 effort=1000.0 velocity=10.0; origin xyz=0.0 0.0 -0.05 rpy=0.0 0.0 0.0 -> xyz=0 0 -0.05 rpy=0 0 0
- joint left_foot_to_left_toes: origin xyz=0.12 0.0 -0.02 rpy=0.0 0.0 0.0 -> xyz=0.12 0 -0.02 rpy=0 0 0
- joint left_shank_to_left_foot_intermediate: origin xyz=0.0 0.0 -0.43 rpy=0.0 0.0 0.0 -> xyz=0 0 -0.43 rpy=0 0 0
- joint left_thigh_to_left_shank: limit lower=0.0 upper=2.62 effort=1000.0 velocity=10.0 -> lower=0 upper=2.62 effort=1000.0 velocity=10.0; origin xyz=0.0 0.0 -0.43 rpy=0.0 0.0 0.0 -> xyz=0 0 -0.43 rpy=0 0 0
- joint lumbar1_to_lumbar2_intermediate: origin xyz=0.0 0.0 0.12 rpy=0.0 0.0 0.0 -> xyz=0 0 0.12 rpy=0 0 0
- joint lumbar2_to_lumbar3_intermediate: origin xyz=0.0 0.0 0.12 rpy=0.0 0.0 0.0 -> xyz=0 0 0.12 rpy=0 0 0
- joint lumbar3_to_thorax1: limit lower=-1.0 upper=1.0 effort=1000.0 velocity=10.0 -> lower=-1 upper=1 effort=1000.0 velocity=10.0; origin xyz=0.0 0.0 0.12 rpy=0.0 0.0 0.0 -> xyz=0 0 0.12 rpy=0 0 0
- joint pelvis_to_left_thigh_gimbal_z: origin xyz=0.0 0.09 -0.05 rpy=0.0 0.0 0.0 -> xyz=0 0.09 -0.05 rpy=0 0 0
- joint pelvis_to_lumbar1_intermediate: origin xyz=0.0 0.0 0.12 rpy=0.0 0.0 0.0 -> xyz=0 0 0.12 rpy=0 0 0
- joint pelvis_to_right_thigh_gimbal_z: origin xyz=0.0 -0.09 -0.05 rpy=0.0 0.0 0.0 -> xyz=0 -0.09 -0.05 rpy=0 0 0
- joint right_foot_to_right_toes: origin xyz=0.12 0.0 -0.02 rpy=0.0 0.0 0.0 -> xyz=0.12 0 -0.02 rpy=0 0 0
- joint right_shank_to_right_foot_intermediate: origin xyz=0.0 0.0 -0.43 rpy=0.0 0.0 0.0 -> xyz=0 0 -0.43 rpy=0 0 0
- joint right_thigh_to_right_shank: limit lower=0.0 upper=2.62 effort=1000.0 velocity=10.0 -> lower=0 upper=2.62 effort=1000.0 velocity=10.0; origin xyz=0.0 0.0 -0.43 rpy=0.0 0.0 0.0 -> xyz=0 0 -0.43 rpy=0 0 0
- joint scapula_left_to_upper_arm_left_gimbal_z: origin xyz=0.0 0.04 0.1 rpy=0.0 0.0 0.0 -> xyz=0 0.04 0.1 rpy=0 0 0
- joint scapula_right_to_upper_arm_right_gimbal_z: origin xyz=0.0 -0.04 0.1 rpy=0.0 0.0 0.0 -> xyz=0 -0.04 0.1 rpy=0 0 0
- joint thorax1_to_thorax2: limit lower=-1.0 upper=1.0 effort=1000.0 velocity=10.0 -> lower=-1 upper=1 effort=1000.0 velocity=10.0; origin xyz=0.0 0.0 0.1 rpy=0.0 0.0 0.0 -> xyz=0 0 0.1 rpy=0 0 0
- joint thorax2_to_thorax3: limit lower=-1.0 upper=1.0 effort=1000.0 velocity=10.0 -> lower=-1 upper=1 effort=1000.0 velocity=10.0; origin xyz=0.0 0.0 0.1 rpy=0.0 0.0 0.0 -> xyz=0 0 0.1 rpy=0 0 0
- joint thorax3_to_scapula_left_intermediate: origin xyz=0.0 0.18 0.28 rpy=0.0 0.0 0.0 -> xyz=0 0.18 0.28 rpy=0 0 0
- joint thorax3_to_scapula_right_intermediate: origin xyz=0.0 -0.18 0.28 rpy=0.0 0.0 0.0 -> xyz=0 -0.18 0.28 rpy=0 0 0
- joint upper_arm_left_to_forearm_left_intermediate: limit lower=0.0 upper=2.62 effort=1000.0 velocity=10.0 -> lower=0 upper=2.62 effort=1000.0 velocity=10.0; origin xyz=0.0 0.0 -0.26 rpy=0.0 0.0 0.0 -> xyz=0 0 -0.26 rpy=0 0 0
- joint upper_arm_right_to_forearm_right_intermediate: limit lower=0.0 upper=2.62 effort=1000.0 velocity=10.0 -> lower=0 upper=2.62 effort=1000.0 velocity=10.0; origin xyz=0.0 0.0 -0.26 rpy=0.0 0.0 0.0 -> xyz=0 0 -0.26 rpy=0 0 0
