Commit message: fix(drake): actuate the golfer URDF so theta reaches the plant (#13421)
The generated Drake golfer URDF declared no <transmission> elements, so
MultibodyPlant built zero actuators. simulate_with_coefficients sized
theta from an nv - 6 fallback (19) but connected the torque source only
when num_actuators() matched, so it never connected: every rollout was
gravity-only while tau logged the command and the status read success.
fit_swing_autodiff used the same fallback.

- humanoid_urdf: emit one SimpleTransmission per revolute joint in URDF
  joint order (19 actuators), and set the joint effort limit to
  ACTUATOR_EFFORT_LIMIT_NM = 1e4 N*m. Drake clamps actuation at the
  limit; the old placeholder 200 N*m would silently clip in-bounds
  theta (POLY_BOUNDS sum to 3225 N*m).
- Regenerate golfer.urdf via build_humanoid_models.py (--check clean)
  and re-pin its sha256 in engine_model_inventory.json.
- simulate: raise when the plant declares no actuators, always connect
  the torque source, and refuse torque beyond the effort limits at the
  discrete plant's step times.
- fit_swing_autodiff: resolve actuators through the same fail-closed
  helper.
- DRAKE_PARITY_SPEC 3.6 records the actuation topology, ordering,
  effort limit, acceptance checks, the torque-free state this replaces,
  limitations and reproduction commands.
- Mocked pydrake harnesses now report per-actuator effort limits, as
  real Drake does.

Co-Authored-By: Claude Opus 5.5 <noreply@anthropic.com>

File: src/engines/physics_engines/drake/models/generated/golfer.urdf (robot description, URDF)
Before this commit: robot golf_humanoid, 22 links, 22 joints
Joints:
- joint left_elbow: limit lower=-2.5 upper=0 effort=200 velocity=20 -> lower=-2.5 upper=0 effort=10000 velocity=20
- joint left_scapula_universal_1: limit lower=-0.5 upper=0.5 effort=200 velocity=20 -> lower=-0.5 upper=0.5 effort=10000 velocity=20
- joint left_scapula_universal_2: limit lower=-0.5 upper=0.5 effort=200 velocity=20 -> lower=-0.5 upper=0.5 effort=10000 velocity=20
- joint left_shoulder_gimbal_1: limit lower=-3.14 upper=3.14 effort=200 velocity=20 -> lower=-3.14 upper=3.14 effort=10000 velocity=20
- joint left_shoulder_gimbal_2: limit lower=-1.5 upper=1.5 effort=200 velocity=20 -> lower=-1.5 upper=1.5 effort=10000 velocity=20
- joint left_shoulder_gimbal_3: limit lower=-1.5 upper=1.5 effort=200 velocity=20 -> lower=-1.5 upper=1.5 effort=10000 velocity=20
- joint left_wrist_universal_1: limit lower=-1 upper=1 effort=200 velocity=20 -> lower=-1 upper=1 effort=10000 velocity=20
- joint left_wrist_universal_2: limit lower=-1 upper=1 effort=200 velocity=20 -> lower=-1 upper=1 effort=10000 velocity=20
- joint right_elbow: limit lower=-2.5 upper=0 effort=200 velocity=20 -> lower=-2.5 upper=0 effort=10000 velocity=20
- joint right_scapula_universal_1: limit lower=-0.5 upper=0.5 effort=200 velocity=20 -> lower=-0.5 upper=0.5 effort=10000 velocity=20
- joint right_scapula_universal_2: limit lower=-0.5 upper=0.5 effort=200 velocity=20 -> lower=-0.5 upper=0.5 effort=10000 velocity=20
- joint right_shoulder_gimbal_1: limit lower=-3.14 upper=3.14 effort=200 velocity=20 -> lower=-3.14 upper=3.14 effort=10000 velocity=20
- joint right_shoulder_gimbal_2: limit lower=-1.5 upper=1.5 effort=200 velocity=20 -> lower=-1.5 upper=1.5 effort=10000 velocity=20
- joint right_shoulder_gimbal_3: limit lower=-1.5 upper=1.5 effort=200 velocity=20 -> lower=-1.5 upper=1.5 effort=10000 velocity=20
- joint right_wrist_universal_1: limit lower=-1 upper=1 effort=200 velocity=20 -> lower=-1 upper=1 effort=10000 velocity=20
- joint right_wrist_universal_2: limit lower=-1 upper=1 effort=200 velocity=20 -> lower=-1 upper=1 effort=10000 velocity=20
- joint spine_twist: limit lower=-1 upper=1 effort=200 velocity=20 -> lower=-1 upper=1 effort=10000 velocity=20
- joint spine_universal_1: limit lower=-0.6 upper=0.6 effort=200 velocity=20 -> lower=-0.6 upper=0.6 effort=10000 velocity=20
- joint spine_universal_2: limit lower=-0.6 upper=0.6 effort=200 velocity=20 -> lower=-0.6 upper=0.6 effort=10000 velocity=20

Commit message: feat(engines): align default models to canonical golfer and raise KeyError on unknown body (#12985) (#13312)
* feat(engines): align default models to canonical golfer and raise KeyError on unknown body (#12985)

* fix(engines): restore MockPhysicsEngine.compute_contact_forces and narrow Drake body enumeration catch (#12985)

The earlier commit on this branch replaced compute_contact_forces with
get_body_names in the mock engine, which broke
test_mock_engine.py::test_compute_contact_forces. Restore it and source
the mock body names from REQUIRED_GOLFER_BODIES (DRY). Replace the blind
except Exception in DrakePhysicsEngine.get_body_names with narrow
exceptions and a debug log, per the error-handling ratchet (BLE001).

Co-Authored-By: Claude Opus 5.5 <noreply@anthropic.com>

* fix(inventory): record regenerated Drake golfer URDF hash and model_contracts in divergence inventory (#12985)

unit-test-gate (1/2) failed on two stale inventories after the Drake URDF
was regenerated from the canonical spec and model_contracts.py was added:
- engine_model_inventory.json drake/legacy-golfer generated_sha256 now
  matches the committed (LF) blob.
- divergence_inventory.v2.jsonl regenerated with
  scripts.shared_tools.divergence_inventory --write (--check passes).

Co-Authored-By: Claude Opus 5.5 <noreply@anthropic.com>

* fix(engines): resolve tools.model_converter under CI PYTHONPATH and bind drake_golfer to canonical links (#12985)

unit-test-gate (2/2) failures:
- test_drake_urdf_no_drift: with PYTHONPATH=.:src, src/ was already on
  sys.path so the script skipped re-inserting it, and the earlier
  src/shared/python insert made tools.model_converter resolve to the
  unrelated src/shared/python/tools package. Always move src/ to the
  front of sys.path.
- test_catalog_imports_bundled_native_urdf_trees: the Drake golfer URDF is
  now generated from the canonical spec, so the legacy DRAKE_LINKS map
  (left_forearm, upper_torso_hub, ...) no longer matches. drake_golfer now
  uses GOLFER_LINKS, and the dead map is removed.

Co-Authored-By: Claude Opus 5.5 <noreply@anthropic.com>

---------

Co-authored-by: Dieter Olson <dieterolson@gmail.com>
Co-authored-by: Claude Opus 5.5 <noreply@anthropic.com>

File: src/engines/physics_engines/drake/models/generated/golfer.urdf (robot description, URDF)
Before this commit: robot golf_humanoid, 22 links, 22 joints
Links:
- removed link left_forearm
- removed link left_hand
- removed link left_hand_left_wrist_universal_dummy_1
- removed link left_scapula_rod
- removed link left_scapula_rod_left_scapula_universal_dummy_1
- removed link left_upper_arm
- removed link left_upper_arm_left_shoulder_gimbal_dummy_1
- removed link left_upper_arm_left_shoulder_gimbal_dummy_2
- removed link lower_spine
- removed link lower_spine_spine_universal_dummy_1
- removed link right_forearm
- removed link right_hand
- removed link right_hand_right_wrist_universal_dummy_1
- removed link right_scapula_rod
- removed link right_scapula_rod_right_scapula_universal_dummy_1
- removed link right_upper_arm
- removed link right_upper_arm_right_shoulder_gimbal_dummy_1
- removed link right_upper_arm_right_shoulder_gimbal_dummy_2
- removed link upper_spine
- removed link upper_torso_hub
- added link club_head, mass 0.23; visual box size=0.12 0.08 0.04
- added link fingers_left, mass 0.2; visual box size=0.05 0.08 0.02
- added link fingers_right, mass 0.2; visual box size=0.05 0.08 0.02
- added link forearm_left, mass 1.5; visual cylinder length=0.13 radius=0.045
- added link forearm_left_intermediate, mass 0.001
- added link forearm_right, mass 1.5; visual cylinder length=0.13 radius=0.045
- added link forearm_right_intermediate, mass 0.001
- added link hand_left, mass 0.5; visual cylinder length=0.095 radius=0.04
- added link hand_left_intermediate, mass 0.001
- added link hand_right, mass 0.5; visual cylinder length=0.095 radius=0.04
- added link hand_right_intermediate, mass 0.001
- added link head, mass 5; visual sphere radius=0.12
- added link left_foot, mass 1.37; visual box size=0.26 0.1 0.07
- added link left_foot_intermediate, mass 0.001
- added link left_shank, mass 3.53; visual cylinder length=0.215 radius=0.05
- added link left_thigh, mass 7.05; visual cylinder length=0.215 radius=0.06
- added link left_thigh_gimbal_y, mass 0.001
- added link left_thigh_gimbal_z, mass 0.001
- added link left_toes, mass 0.3; visual box size=0.1 0.08 0.03
- added link lumbar1, mass 2; visual cylinder length=0.12 radius=0.08
- added link lumbar1_intermediate, mass 0.001
- added link lumbar2, mass 2; visual cylinder length=0.12 radius=0.08
- added link lumbar2_intermediate, mass 0.001
- added link lumbar3, mass 2; visual cylinder length=0.12 radius=0.08
- added link lumbar3_intermediate, mass 0.001
- added link mid_hands
- added link right_foot, mass 1.37; visual box size=0.26 0.1 0.07
- added link right_foot_intermediate, mass 0.001
- added link right_shank, mass 3.53; visual cylinder length=0.215 radius=0.05
- added link right_thigh, mass 7.05; visual cylinder length=0.215 radius=0.06
- added link right_thigh_gimbal_y, mass 0.001
- added link right_thigh_gimbal_z, mass 0.001
- added link right_toes, mass 0.3; visual box size=0.1 0.08 0.03
- added link scapula_left, mass 1.5; visual box size=0.12 0.08 0.05
- added link scapula_left_intermediate, mass 0.001
- added link scapula_right, mass 1.5; visual box size=0.12 0.08 0.05
- added link scapula_right_intermediate, mass 0.001
- added link thorax1, mass 6; visual cylinder length=0.1 radius=0.08
- added link thorax2, mass 6; visual cylinder length=0.1 radius=0.08
- added link thorax3, mass 6; visual cylinder length=0.1 radius=0.08
- added link upper_arm_left, mass 2.5; visual cylinder length=0.14 radius=0.05
- added link upper_arm_left_gimbal_y, mass 0.001
- added link upper_arm_left_gimbal_z, mass 0.001
- added link upper_arm_right, mass 2.5; visual cylinder length=0.14 radius=0.05
- added link upper_arm_right_gimbal_y, mass 0.001
- added link upper_arm_right_gimbal_z, mass 0.001
- link club_shaft: mass 0.4 -> 0.12; geometry visual cylinder length=0.5 radius=0.015
- link pelvis: mass 12 -> 11.7; geometry visual cylinder length=0.2 radius=0.15
Joints:
- removed joint grip_lead
- removed joint left_elbow
- removed joint left_scapula_universal_1
- removed joint left_scapula_universal_2
- removed joint left_shoulder_gimbal_1
- removed joint left_shoulder_gimbal_2
- removed joint left_shoulder_gimbal_3
- removed joint left_wrist_universal_1
- removed joint left_wrist_universal_2
- removed joint pelvis_floating
- removed joint right_elbow
- removed joint right_scapula_universal_1
- removed joint right_scapula_universal_2
- removed joint right_shoulder_gimbal_1
- removed joint right_shoulder_gimbal_2
- removed joint right_shoulder_gimbal_3
- removed joint right_wrist_universal_1
- removed joint right_wrist_universal_2
- removed joint spine_twist
- removed joint spine_universal_1
- removed joint spine_universal_2
- removed joint torso_weld
- added joint club_shaft_to_club_head: type fixed, parent club_shaft, child club_head, origin xyz=0 0 -0.5 rpy=0 0 0
- added joint forearm_left_intermediate_to_forearm_left: type revolute, parent forearm_left_intermediate, child forearm_left, origin xyz=0.0 0.0 0.0 rpy=0.0 0.0 0.0, axis 1 0 0, limit lower=-1.57 upper=1.57 effort=1000.0 velocity=10.0
- added joint forearm_left_to_hand_left_intermediate: type revolute, parent forearm_left, child hand_left_intermediate, origin xyz=0 0 -0.19 rpy=0 0 0, axis 0 1 0, limit lower=-1.22 upper=1.22 effort=1000.0 velocity=10.0
- added joint forearm_right_intermediate_to_forearm_right: type revolute, parent forearm_right_intermediate, child forearm_right, origin xyz=0.0 0.0 0.0 rpy=0.0 0.0 0.0, axis 1 0 0, limit lower=-1.57 upper=1.57 effort=1000.0 velocity=10.0
- added joint forearm_right_to_hand_right_intermediate: type revolute, parent forearm_right, child hand_right_intermediate, origin xyz=0 0 -0.19 rpy=0 0 0, axis 0 1 0, limit lower=-1.22 upper=1.22 effort=1000.0 velocity=10.0
- added joint hand_left_intermediate_to_hand_left: type revolute, parent hand_left_intermediate, child hand_left, origin xyz=0.0 0.0 0.0 rpy=0.0 0.0 0.0, axis 0 0 1, limit lower=-0.52 upper=0.7 effort=1000.0 velocity=10.0
- added joint hand_left_to_fingers_left: type revolute, parent hand_left, child fingers_left, origin xyz=0 0 -0.05 rpy=0 0 0, axis 0 1 0, limit lower=0 upper=1.57 effort=1000.0 velocity=10.0
- added joint hand_right_intermediate_to_hand_right: type revolute, parent hand_right_intermediate, child hand_right, origin xyz=0.0 0.0 0.0 rpy=0.0 0.0 0.0, axis 0 0 1, limit lower=-0.52 upper=0.7 effort=1000.0 velocity=10.0
- added joint hand_right_to_fingers_right: type revolute, parent hand_right, child fingers_right, origin xyz=0 0 -0.05 rpy=0 0 0, axis 0 1 0, limit lower=0 upper=1.57 effort=1000.0 velocity=10.0
- added joint left_foot_intermediate_to_left_foot: type revolute, parent left_foot_intermediate, child left_foot, origin xyz=0.0 0.0 0.0 rpy=0.0 0.0 0.0, axis 0 1 0, limit lower=-0.35 upper=0.35 effort=1000.0 velocity=10.0
- added joint left_foot_to_left_toes: type revolute, parent left_foot, child left_toes, origin xyz=0.12 0 -0.02 rpy=0 0 0, axis 0 1 0, limit lower=-0.35 upper=0.52 effort=1000.0 velocity=10.0
- added joint left_shank_to_left_foot_intermediate: type revolute, parent left_shank, child left_foot_intermediate, origin xyz=0 0 -0.43 rpy=0 0 0, axis 1 0 0, limit lower=-0.7 upper=0.52 effort=1000.0 velocity=10.0
- added joint left_thigh_gimbal_y_to_left_thigh: type revolute, parent left_thigh_gimbal_y, child left_thigh, origin xyz=0.0 0.0 0.0 rpy=0.0 0.0 0.0, axis 0 0 1, limit lower=-0.7 upper=0.7 effort=1000.0 velocity=10.0
- added joint left_thigh_gimbal_z_to_left_thigh_gimbal_y: type revolute, parent left_thigh_gimbal_z, child left_thigh_gimbal_y, origin xyz=0.0 0.0 0.0 rpy=0.0 0.0 0.0, axis 1 0 0, limit lower=-0.87 upper=0.52 effort=1000.0 velocity=10.0
- added joint left_thigh_to_left_shank: type revolute, parent left_thigh, child left_shank, origin xyz=0 0 -0.43 rpy=0 0 0, axis 0 1 0, limit lower=0 upper=2.62 effort=1000.0 velocity=10.0
- added joint lumbar1_intermediate_to_lumbar1: type revolute, parent lumbar1_intermediate, child lumbar1, origin xyz=0.0 0.0 0.0 rpy=0.0 0.0 0.0, axis 0 1 0, limit lower=-0.35 upper=0.35 effort=1000.0 velocity=10.0
- added joint lumbar1_to_lumbar2_intermediate: type revolute, parent lumbar1, child lumbar2_intermediate, origin xyz=0 0 0.12 rpy=0 0 0, axis 1 0 0, limit lower=-0.7 upper=0.52 effort=1000.0 velocity=10.0
- added joint lumbar2_intermediate_to_lumbar2: type revolute, parent lumbar2_intermediate, child lumbar2, origin xyz=0.0 0.0 0.0 rpy=0.0 0.0 0.0, axis 0 1 0, limit lower=-0.35 upper=0.35 effort=1000.0 velocity=10.0
- added joint lumbar2_to_lumbar3_intermediate: type revolute, parent lumbar2, child lumbar3_intermediate, origin xyz=0 0 0.12 rpy=0 0 0, axis 1 0 0, limit lower=-0.7 upper=0.52 effort=1000.0 velocity=10.0
- added joint lumbar3_intermediate_to_lumbar3: type revolute, parent lumbar3_intermediate, child lumbar3, origin xyz=0.0 0.0 0.0 rpy=0.0 0.0 0.0, axis 0 1 0, limit lower=-0.35 upper=0.35 effort=1000.0 velocity=10.0
- added joint lumbar3_to_thorax1: type revolute, parent lumbar3, child thorax1, origin xyz=0 0 0.12 rpy=0 0 0, axis 0 0 1, limit lower=-1 upper=1 effort=1000.0 velocity=10.0
- added joint mid_hands_to_club_shaft: type fixed, parent mid_hands, child club_shaft, origin xyz=0.0 0.0 -0.05 rpy=0.0 0.0 0.0
- added joint pelvis_to_left_thigh_gimbal_z: type revolute, parent pelvis, child left_thigh_gimbal_z, origin xyz=0 0.09 -0.05 rpy=0 0 0, axis 0 1 0, limit lower=-1.57 upper=1.57 effort=1000.0 velocity=10.0
- added joint pelvis_to_lumbar1_intermediate: type revolute, parent pelvis, child lumbar1_intermediate, origin xyz=0 0 0.12 rpy=0 0 0, axis 1 0 0, limit lower=-0.7 upper=0.52 effort=1000.0 velocity=10.0
- added joint pelvis_to_right_thigh_gimbal_z: type revolute, parent pelvis, child right_thigh_gimbal_z, origin xyz=0 -0.09 -0.05 rpy=0 0 0, axis 0 1 0, limit lower=-1.57 upper=1.57 effort=1000.0 velocity=10.0
- added joint right_foot_intermediate_to_right_foot: type revolute, parent right_foot_intermediate, child right_foot, origin xyz=0.0 0.0 0.0 rpy=0.0 0.0 0.0, axis 0 1 0, limit lower=-0.35 upper=0.35 effort=1000.0 velocity=10.0
- added joint right_foot_to_right_toes: type revolute, parent right_foot, child right_toes, origin xyz=0.12 0 -0.02 rpy=0 0 0, axis 0 1 0, limit lower=-0.35 upper=0.52 effort=1000.0 velocity=10.0
- added joint right_shank_to_right_foot_intermediate: type revolute, parent right_shank, child right_foot_intermediate, origin xyz=0 0 -0.43 rpy=0 0 0, axis 1 0 0, limit lower=-0.7 upper=0.52 effort=1000.0 velocity=10.0
- added joint right_thigh_gimbal_y_to_right_thigh: type revolute, parent right_thigh_gimbal_y, child right_thigh, origin xyz=0.0 0.0 0.0 rpy=0.0 0.0 0.0, axis 0 0 1, limit lower=-0.7 upper=0.7 effort=1000.0 velocity=10.0
- added joint right_thigh_gimbal_z_to_right_thigh_gimbal_y: type revolute, parent right_thigh_gimbal_z, child right_thigh_gimbal_y, origin xyz=0.0 0.0 0.0 rpy=0.0 0.0 0.0, axis 1 0 0, limit lower=-0.87 upper=0.52 effort=1000.0 velocity=10.0
- added joint right_thigh_to_right_shank: type revolute, parent right_thigh, child right_shank, origin xyz=0 0 -0.43 rpy=0 0 0, axis 0 1 0, limit lower=0 upper=2.62 effort=1000.0 velocity=10.0
- added joint scapula_left_intermediate_to_scapula_left: type revolute, parent scapula_left_intermediate, child scapula_left, origin xyz=0.0 0.0 0.0 rpy=0.0 0.0 0.0, axis 0 1 0, limit lower=-0.52 upper=0.52 effort=1000.0 velocity=10.0
- added joint scapula_left_to_upper_arm_left_gimbal_z: type revolute, parent scapula_left, child upper_arm_left_gimbal_z, origin xyz=0 0.04 0.1 rpy=0 0 0, axis 0 1 0, limit lower=-1.57 upper=3.1416 effort=1000.0 velocity=10.0
- added joint scapula_right_intermediate_to_scapula_right: type revolute, parent scapula_right_intermediate, child scapula_right, origin xyz=0.0 0.0 0.0 rpy=0.0 0.0 0.0, axis 0 1 0, limit lower=-0.52 upper=0.52 effort=1000.0 velocity=10.0
- added joint scapula_right_to_upper_arm_right_gimbal_z: type revolute, parent scapula_right, child upper_arm_right_gimbal_z, origin xyz=0 -0.04 0.1 rpy=0 0 0, axis 0 1 0, limit lower=-1.57 upper=3.1416 effort=1000.0 velocity=10.0
- added joint thorax1_to_thorax2: type revolute, parent thorax1, child thorax2, origin xyz=0 0 0.1 rpy=0 0 0, axis 0 0 1, limit lower=-1 upper=1 effort=1000.0 velocity=10.0
- added joint thorax2_to_thorax3: type revolute, parent thorax2, child thorax3, origin xyz=0 0 0.1 rpy=0 0 0, axis 0 0 1, limit lower=-1 upper=1 effort=1000.0 velocity=10.0
- added joint thorax3_to_head: type fixed, parent thorax3, child head, origin xyz=0 0 0.15 rpy=0 0 0
- added joint thorax3_to_mid_hands: type fixed, parent thorax3, child mid_hands, origin xyz=0.0 0.0 -0.17 rpy=0.0 0.0 0.0
- added joint thorax3_to_scapula_left_intermediate: type revolute, parent thorax3, child scapula_left_intermediate, origin xyz=0 0.18 0.28 rpy=0 0 0, axis 0 0 1, limit lower=-0.35 upper=0.7 effort=1000.0 velocity=10.0
- added joint thorax3_to_scapula_right_intermediate: type revolute, parent thorax3, child scapula_right_intermediate, origin xyz=0 -0.18 0.28 rpy=0 0 0, axis 0 0 1, limit lower=-0.35 upper=0.7 effort=1000.0 velocity=10.0
- added joint upper_arm_left_gimbal_y_to_upper_arm_left: type revolute, parent upper_arm_left_gimbal_y, child upper_arm_left, origin xyz=0.0 0.0 0.0 rpy=0.0 0.0 0.0, axis 0 0 1, limit lower=-1.57 upper=1.57 effort=1000.0 velocity=10.0
- added joint upper_arm_left_gimbal_z_to_upper_arm_left_gimbal_y: type revolute, parent upper_arm_left_gimbal_z, child upper_arm_left_gimbal_y, origin xyz=0.0 0.0 0.0 rpy=0.0 0.0 0.0, axis 1 0 0, limit lower=-0.52 upper=2.09 effort=1000.0 velocity=10.0
- added joint upper_arm_left_to_forearm_left_intermediate: type revolute, parent upper_arm_left, child forearm_left_intermediate, origin xyz=0 0 -0.26 rpy=0 0 0, axis 0 1 0, limit lower=0 upper=2.62 effort=1000.0 velocity=10.0
- added joint upper_arm_right_gimbal_y_to_upper_arm_right: type revolute, parent upper_arm_right_gimbal_y, child upper_arm_right, origin xyz=0.0 0.0 0.0 rpy=0.0 0.0 0.0, axis 0 0 1, limit lower=-1.57 upper=1.57 effort=1000.0 velocity=10.0
- added joint upper_arm_right_gimbal_z_to_upper_arm_right_gimbal_y: type revolute, parent upper_arm_right_gimbal_z, child upper_arm_right_gimbal_y, origin xyz=0.0 0.0 0.0 rpy=0.0 0.0 0.0, axis 1 0 0, limit lower=-0.52 upper=2.09 effort=1000.0 velocity=10.0
- added joint upper_arm_right_to_forearm_right_intermediate: type revolute, parent upper_arm_right, child forearm_right_intermediate, origin xyz=0 0 -0.26 rpy=0 0 0, axis 0 1 0, limit lower=0 upper=2.62 effort=1000.0 velocity=10.0
